Commit message: add handi simulation

File: denso_robot_descriptions/robots/cobotta/urdf/denso_robot.ros2_control.xacro (robot description, xacro)
@@ -13,6 +13,6 @@
     ">
     <ros2_control name="${namespace}${name}" type="system">
-	<!-- joint limits include -->
-	<xacro:include filename="$(find denso_robot_descriptions)/robots/$(arg model)/urdf/denso_robot_joint_limits.xacro" />
+      <!-- joint limits include -->
+      <xacro:include filename="$(find denso_robot_descriptions)/robots/$(arg model)/urdf/denso_robot_joint_limits.xacro" />
       <hardware>
         <xacro:if value="${sim}">

File: denso_robot_descriptions/robots/cobotta/urdf/denso_robot_kinematics.xacro (robot description, xacro)
@@ -207,11 +207,35 @@
 			</inertial>
 		</link>
-		<joint name="$(arg namespace)joint_gripper" type="revolute">
+		<joint name="$(arg namespace)joint_gripper" type="fixed">
 			<parent link="$(arg namespace)J6"/>
 			<child link="$(arg namespace)gripper_base"/>
 			<origin rpy="0.000000 0.000000 0.000000" xyz="0.000000 0.0 0.0001"/>
 			<axis xyz="-0.000000 -0.000000 1.000000"/>
-			<limit effort="1" lower="-3.1415926575" upper="3.1415926575" velocity="3.83012504350156"/>
-			<dynamics damping="0" friction="0"/>
+		</joint>
+		<link name="$(arg namespace)left_finger">
+			<visual>
+				<origin rpy="0 0 0" xyz="0 0 0"/>
+				<geometry>
+					<mesh filename="file:///$(find denso_robot_descriptions)/robots/$(arg model)/meshes/left_finger.dae" scale="1 1 1"/>
+				</geometry>
+			</visual>
+			<collision>
+				<origin rpy="0 0 0" xyz="0 0 0"/>
+				<geometry>
+					<mesh filename="file:///$(find denso_robot_descriptions)/robots/$(arg model)/meshes/left_finger.dae" scale="1 1 1"/>
+				</geometry>
+			</collision>
+			<inertial>
+				<mass value="1"/>
+				<origin rpy="0.000000 0.000000 0.000000" xyz="0.000000 0.000000 0.000000"/>
+				<inertia ixx="1" ixy="0" ixz="0" iyy="1" iyz="0" izz="1"/>
+			</inertial>
+		</link>
+		<joint name="$(arg namespace)cobotta_finger_joint1" type="prismatic">
+			<parent link="$(arg namespace)gripper_base"/>
+			<child link="$(arg namespace)left_finger"/>
+			<origin rpy="0.000000 0.000000 0.000000" xyz="0.000000 0.0001 0.000"/>
+			<axis xyz="0.000000 1.000000 0.000000"/>
+			<limit effort="20" lower="0.0" upper="0.015" velocity="0.15"/>
 		</joint>
 		<link name="$(arg namespace)right_finger">
@@ -234,39 +258,17 @@
 			</inertial>
 		</link>
-		<joint name="$(arg namespace)joint_right_finger" type="prismatic">
+		<joint name="$(arg namespace)cobotta_finger_joint2" type="prismatic">
+			<mimic joint="cobotta_finger_joint1" multiplier="-1" offset="0" />
 			<parent link="$(arg namespace)gripper_base"/>
 			<child link="$(arg namespace)right_finger"/>
 			<origin rpy="0.000000 0.000000 0.000000" xyz="0.000000 -0.0001 0.000"/>
 			<axis xyz="0.000000 1.000000 0.000000"/>
-			<limit effort="1" lower="-0.015" upper="0.0" velocity="0.015"/>
-			<dynamics damping="0" friction="0"/>
-		</joint>
-		<link name="$(arg namespace)left_finger">
-			<visual>
-				<origin rpy="0 0 0" xyz="0 0 0"/>
-				<geometry>
-					<mesh filename="file:///$(find denso_robot_descriptions)/robots/$(arg model)/meshes/left_finger.dae" scale="1 1 1"/>
-				</geometry>
-			</visual>
-			<collision>
-				<origin rpy="0 0 0" xyz="0 0 0"/>
-				<geometry>
-					<mesh filename="file:///$(find denso_robot_descriptions)/robots/$(arg model)/meshes/left_finger.dae" scale="1 1 1"/>
-				</geometry>
-			</collision>
-			<inertial>
-				<mass value="1"/>
-				<origin rpy="0.000000 0.000000 0.000000" xyz="0.000000 0.000000 0.000000"/>
-				<inertia ixx="1" ixy="0" ixz="0" iyy="1" iyz="0" izz="1"/>
-			</inertial>
-		</link>
-		<joint name="$(arg namespace)joint_left_finger" type="prismatic">
-			<parent link="$(arg namespace)gripper_base"/>
-			<child link="$(arg namespace)left_finger"/>
-			<origin rpy="0.000000 0.000000 0.000000" xyz="0.000000 0.0001 0.000"/>
-			<axis xyz="0.000000 1.000000 0.000000"/>
-			<limit effort="1" lower="0.0" upper="0.015" velocity="0.015"/>
-			<dynamics damping="0" friction="0"/>
-		</joint>
+			<limit effort="5" lower="-0.015" upper="0.0" velocity="0.2"/>
+		</joint>
+		<joint name="$(arg namespace)cobotta_finger_joint2_mimic" type="fixed">
+			<parent link="world" />
+			<child link="random" />
+		</joint>
+		<link name="random"/>
 	</xacro:macro>
 </robot>

File: denso_robot_descriptions/robots/cobotta/urdf/denso_robot_macro.xacro (robot description, xacro)
@@ -63,7 +63,12 @@
     <!-- links -  main serial chain -->
     <xacro:denso_robot_arm_kinematics namespace="$(arg namespace)" model="$(arg model)" />
+    <!-- For Simulation     -->
+    <xacro:if value="${sim}">
+      <xacro:include filename="$(find denso_robot_descriptions)/robots/$(arg model)/urdf/denso_robot_hand.ros2_control.xacro" />
+      <xacro:cobotta_hand_ros2_control name="GazeboHandSystem" ros2_control_hardware_type="gazebo" />
+    </xacro:if>
     <gazebo>
       <plugin filename="libgazebo_ros2_control.so" name="gazebo_ros2_control">
-  	    <parameters>$(find denso_robot_moveit_config)/robots/$(arg model)/config/denso_robot_controllers.yaml</parameters>
+  	    <parameters>$(find denso_robot_moveit_config)/robots/$(arg model)/config/denso_robot_controllers_gazebo.yaml</parameters>
       </plugin>
     </gazebo>

File: denso_robot_moveit_config/robots/cobotta/srdf/denso_robot_macro.srdf.xacro (robot description, xacro)
@@ -20,7 +20,9 @@
 	  </group>
     <group name="${namespace}hand">
-		<joint name="$(arg namespace)joint_gripper"/>
-		<joint name="$(arg namespace)joint_right_finger"/>
-		<joint name="$(arg namespace)joint_left_finger"/>
+	    <link name="$(arg namespace)gripper_base" />
+      	<link name="$(arg namespace)left_finger" />
+      	<link name="$(arg namespace)right_finger" />
+		<joint name="$(arg namespace)cobotta_finger_joint1" />
+		<joint name="$(arg namespace)cobotta_finger_joint2" />
 	  </group>
     <!--GROUP STATES - Purpose - Define a named state for a particular group, in terms of joint values. This is useful to define states like 'folded arms'-->
@@ -38,6 +40,7 @@
 	<disable_collisions link1="$(arg namespace)J4" link2="$(arg namespace)J5" reason="Adjacent"/>
 	<disable_collisions link1="$(arg namespace)J6" link2="$(arg namespace)gripper_base" reason="Adjacent"/>
-  <disable_collisions link1="$(arg namespace)gripper_base" link2="$(arg namespace)right_finger" reason="Adjacent"/>
-  <disable_collisions link1="$(arg namespace)gripper_base" link2="$(arg namespace)left_finger" reason="Adjacent"/>
+  	<disable_collisions link1="$(arg namespace)gripper_base" link2="$(arg namespace)right_finger" reason="Adjacent"/>
+ 	<disable_collisions link1="$(arg namespace)gripper_base" link2="$(arg namespace)left_finger" reason="Adjacent"/>
+	<disable_collisions link1="$(arg namespace)right_finger" link2="$(arg namespace)left_finger" reason="Default"/>
   </xacro:macro>
 </robot>
