Commit message: try to add hand controller:: debugging...

File: denso_robot_descriptions/robots/cobotta/urdf/denso_robot_hand.ros2_control.xacro (robot description, xacro)
@@ -7,4 +7,15 @@
                     <plugin>gazebo_ros2_control/GazeboSystem</plugin>
                 </xacro:if>
+                <xacro:if value="${ros2_control_hardware_type == 'cobotta'}">
+                    <plugin>denso_robot_control/CobottaHandHW</plugin>
+                    <param name="robot_name">CVR038A1</param>
+                    <param name="ip_address">127.0.0.1</param>
+                    <param name="node_name">denso_hand_controller</param>
+                    <param name="node_namespace">cobotta</param>
+                    <param name="joint">cobotta_finger_joint1</param>
+                    <param name="send_format">0</param>
+                    <param name="recv_format">2</param>
+                    <param name="verbose">true</param>
+                </xacro:if>
                 <xacro:if value="${ros2_control_hardware_type == 'isaac'}">
                     <plugin>topic_based_ros2_control/TopicBasedSystem</plugin>
@@ -13,23 +24,49 @@
                 </xacro:if>
             </hardware>
-            <joint name="cobotta_finger_joint1">
-                <command_interface name="position" />
-                <state_interface name="position">
-                  <param name="initial_value">0.0</param>
-                </state_interface>
-                <state_interface name="velocity">
+            <xacro:if value="${ros2_control_hardware_type == 'gazebo'}">
+                <joint name="cobotta_finger_joint1">
+                    <command_interface name="position" />
+                    <state_interface name="position">
                     <param name="initial_value">0.0</param>
-                </state_interface>
-            </joint>
-            <joint name="cobotta_finger_joint2">
-                <param name="mimic">cobotta_finger_joint1</param>
-                <param name="multiplier">-1</param>
-                <state_interface name="position">
-                  <param name="initial_value">0.0</param>
-                </state_interface>
-                <state_interface name="velocity">
+                    </state_interface>
+                    <state_interface name="velocity">
+                        <param name="initial_value">0.0</param>
+                    </state_interface>
+                </joint>
+                <joint name="cobotta_finger_joint2">
+                    <param name="mimic">cobotta_finger_joint1</param>
+                    <param name="multiplier">-1</param>
+                    <state_interface name="position">
                     <param name="initial_value">0.0</param>
-                </state_interface>
-            </joint>
+                    </state_interface>
+                    <state_interface name="velocity">
+                        <param name="initial_value">0.0</param>
+                    </state_interface>
+                </joint>
+            </xacro:if>
+            <xacro:if value="${ros2_control_hardware_type == 'cobotta'}">
+            <!--     -->
+                <joint name="cobotta_finger_joint1">
+                    <command_interface name="position" />
+                    <state_interface name="position">
+                    <param name="initial_value">0.015</param>
+                    </state_interface>
+                    <state_interface name="velocity">
+                        <param name="initial_value">0.0</param>
+                    </state_interface>
+                </joint>
+                <!--
+                <joint name="cobotta_finger_joint2">
+                    <param name="mimic">cobotta_finger_joint1</param>
+                    <param name="multiplier">-1</param>
+                    <state_interface name="position">
+                    <param name="initial_value">0.0</param>
+                    </state_interface>
+                    <state_interface name="velocity">
+                        <param name="initial_value">0.0</param>
+                    </state_interface>
+                </joint>
+                -->
+            </xacro:if>
         </ros2_control>
     </xacro:macro>

File: denso_robot_descriptions/robots/cobotta/urdf/denso_robot_macro.xacro (robot description, xacro)
@@ -64,8 +64,11 @@
     <xacro:denso_robot_arm_kinematics namespace="$(arg namespace)" model="$(arg model)" />
     <!-- For Simulation     -->
+    <xacro:include filename="$(find denso_robot_descriptions)/robots/$(arg model)/urdf/denso_robot_hand.ros2_control.xacro" />
     <xacro:if value="${sim}">
-      <xacro:include filename="$(find denso_robot_descriptions)/robots/$(arg model)/urdf/denso_robot_hand.ros2_control.xacro" />
       <xacro:cobotta_hand_ros2_control name="GazeboHandSystem" ros2_control_hardware_type="gazebo" />
     </xacro:if>
+    <xacro:unless value="${sim}">
+      <xacro:cobotta_hand_ros2_control name="CobottaHandSystem" ros2_control_hardware_type="cobotta" />
+    </xacro:unless>
     <gazebo>
       <plugin filename="libgazebo_ros2_control.so" name="gazebo_ros2_control">

Commit message: Update cobotta hand controller

File: denso_robot_descriptions/robots/cobotta/urdf/denso_robot_hand.ros2_control.xacro (robot description, xacro)
@@ -1,28 +1,23 @@
 <?xml version="1.0"?>
 <robot xmlns:xacro="http://www.ros.org/wiki/xacro">
-    <xacro:macro name="cobotta_hand_ros2_control" params="name ros2_control_hardware_type">
+    <xacro:macro name="cobotta_hand_ros2_control" params="name namespace sim ip_address verbose">
         <ros2_control name="${name}" type="system">
             <hardware>
-                <xacro:if value="${ros2_control_hardware_type == 'gazebo'}">
+                <xacro:if value="${sim}">
                     <plugin>gazebo_ros2_control/GazeboSystem</plugin>
                 </xacro:if>
-                <xacro:if value="${ros2_control_hardware_type == 'cobotta'}">
+                <xacro:unless value="${sim}">
                     <plugin>denso_robot_control/CobottaHandHW</plugin>
                     <param name="robot_name">CVR038A1</param>
-                    <param name="ip_address">127.0.0.1</param>
+                    <param name="ip_address">${ip_address}</param>
                     <param name="node_name">denso_hand_controller</param>
-                    <param name="node_namespace">cobotta</param>
+                    <param name="node_namespace">${namespace}cobotta</param>
                     <param name="joint">cobotta_finger_joint1</param>
                     <param name="send_format">0</param>
                     <param name="recv_format">2</param>
-                    <param name="verbose">true</param>
-                </xacro:if>
-                <xacro:if value="${ros2_control_hardware_type == 'isaac'}">
-                    <plugin>topic_based_ros2_control/TopicBasedSystem</plugin>
-                    <param name="joint_commands_topic">/isaac_joint_commands</param>
-                    <param name="joint_states_topic">/isaac_joint_states</param>
-                </xacro:if>
+                    <param name="verbose">${verbose}</param>
+                </xacro:unless>
             </hardware>
-            <xacro:if value="${ros2_control_hardware_type == 'gazebo'}">
+            <xacro:if value="${sim}">
                 <joint name="cobotta_finger_joint1">
                     <command_interface name="position" />
@@ -45,6 +40,5 @@
                 </joint>
             </xacro:if>
-            <xacro:if value="${ros2_control_hardware_type == 'cobotta'}">
-            <!--     -->
+            <xacro:unless value="${sim}">
                 <joint name="cobotta_finger_joint1">
                     <command_interface name="position" />
@@ -56,17 +50,5 @@
                     </state_interface>
                 </joint>
-                <!--
-                <joint name="cobotta_finger_joint2">
-                    <param name="mimic">cobotta_finger_joint1</param>
-                    <param name="multiplier">-1</param>
-                    <state_interface name="position">
-                    <param name="initial_value">0.0</param>
-                    </state_interface>
-                    <state_interface name="velocity">
-                        <param name="initial_value">0.0</param>
-                    </state_interface>
-                </joint>
-                -->
-            </xacro:if>
+            </xacro:unless>
         </ros2_control>
     </xacro:macro>

File: denso_robot_descriptions/robots/cobotta/urdf/denso_robot_macro.xacro (robot description, xacro)
@@ -65,10 +65,6 @@
     <!-- For Simulation     -->
     <xacro:include filename="$(find denso_robot_descriptions)/robots/$(arg model)/urdf/denso_robot_hand.ros2_control.xacro" />
-    <xacro:if value="${sim}">
-      <xacro:cobotta_hand_ros2_control name="GazeboHandSystem" ros2_control_hardware_type="gazebo" />
-    </xacro:if>
-    <xacro:unless value="${sim}">
-      <xacro:cobotta_hand_ros2_control name="CobottaHandSystem" ros2_control_hardware_type="cobotta" />
-    </xacro:unless>
+    <xacro:cobotta_hand_ros2_control name="CobottaHandSystem" namespace="$(arg namespace)"
+      sim="$(arg sim)" ip_address="$(arg ip_address)" verbose="$(arg verbose)" />
     <gazebo>
       <plugin filename="libgazebo_ros2_control.so" name="gazebo_ros2_control">
