Commit message: add finger

File: denso_robot_descriptions/robots/cobotta/urdf/denso_robot_kinematics.xacro (robot description, xacro)
@@ -188,4 +188,85 @@
 			<dynamics damping="0" friction="0"/>
 		</joint>
+		<link name="$(arg namespace)gripper_base">
+			<visual>
+				<origin rpy="0 0 0" xyz="0.0 0 0"/>
+				<geometry>
+					<mesh filename="file:///$(find denso_robot_descriptions)/robots/$(arg model)/meshes/gripper_base.dae" scale="1 1 1"/>
+				</geometry>
+			</visual>
+			<collision>
+				<origin rpy="0 0 0" xyz="0 0 0"/>
+				<geometry>
+					<mesh filename="file:///$(find denso_robot_descriptions)/robots/$(arg model)/meshes/gripper_base.dae" scale="1 1 1"/>
+				</geometry>
+			</collision>
+			<inertial>
+				<mass value="1"/>
+				<origin rpy="0.000000 0.000000 0.000000" xyz="0.000000 0.000000 0.000000"/>
+				<inertia ixx="1" ixy="0" ixz="0" iyy="1" iyz="0" izz="1"/>
+			</inertial>
+		</link>
+		<joint name="$(arg namespace)joint_gripper" type="revolute">
+			<parent link="$(arg namespace)J6"/>
+			<child link="$(arg namespace)gripper_base"/>
+			<origin rpy="0.000000 0.000000 0.000000" xyz="0.000000 0.0 0.0001"/>
+			<axis xyz="-0.000000 -0.000000 1.000000"/>
+			<limit effort="1" lower="-3.1415926575" upper="3.1415926575" velocity="3.83012504350156"/>
+			<dynamics damping="0" friction="0"/>
+		</joint>
+		<link name="$(arg namespace)right_finger">
+			<visual>
+				<origin rpy="0 0 0" xyz="0 0 0"/>
+				<geometry>
+					<mesh filename="file:///$(find denso_robot_descriptions)/robots/$(arg model)/meshes/right_finger.dae" scale="1 1 1"/>
+				</geometry>
+			</visual>
+			<collision>
+				<origin rpy="0 0 0" xyz="0 0 0"/>
+				<geometry>
+					<mesh filename="file:///$(find denso_robot_descriptions)/robots/$(arg model)/meshes/right_finger.dae" scale="1 1 1"/>
+				</geometry>
+			</collision>
+			<inertial>
+				<mass value="1"/>
+				<origin rpy="0.000000 0.000000 0.000000" xyz="0.000000 0.000000 0.000000"/>
+				<inertia ixx="1" ixy="0" ixz="0" iyy="1" iyz="0" izz="1"/>
+			</inertial>
+		</link>
+		<joint name="$(arg namespace)joint_right_finger" type="prismatic">
+			<parent link="$(arg namespace)gripper_base"/>
+			<child link="$(arg namespace)right_finger"/>
+			<origin rpy="0.000000 0.000000 0.000000" xyz="0.000000 -0.0001 0.000"/>
+			<axis xyz="0.000000 1.000000 0.000000"/>
+			<limit effort="1" lower="-0.015" upper="0.0" velocity="0.015"/>
+			<dynamics damping="0" friction="0"/>
+		</joint>
+		<link name="$(arg namespace)left_finger">
+			<visual>
+				<origin rpy="0 0 0" xyz="0 0 0"/>
+				<geometry>
+					<mesh filename="file:///$(find denso_robot_descriptions)/robots/$(arg model)/meshes/left_finger.dae" scale="1 1 1"/>
+				</geometry>
+			</visual>
+			<collision>
+				<origin rpy="0 0 0" xyz="0 0 0"/>
+				<geometry>
+					<mesh filename="file:///$(find denso_robot_descriptions)/robots/$(arg model)/meshes/left_finger.dae" scale="1 1 1"/>
+				</geometry>
+			</collision>
+			<inertial>
+				<mass value="1"/>
+				<origin rpy="0.000000 0.000000 0.000000" xyz="0.000000 0.000000 0.000000"/>
+				<inertia ixx="1" ixy="0" ixz="0" iyy="1" iyz="0" izz="1"/>
+			</inertial>
+		</link>
+		<joint name="$(arg namespace)joint_left_finger" type="prismatic">
+			<parent link="$(arg namespace)gripper_base"/>
+			<child link="$(arg namespace)left_finger"/>
+			<origin rpy="0.000000 0.000000 0.000000" xyz="0.000000 0.0001 0.000"/>
+			<axis xyz="0.000000 1.000000 0.000000"/>
+			<limit effort="1" lower="0.0" upper="0.015" velocity="0.015"/>
+			<dynamics damping="0" friction="0"/>
+		</joint>
 	</xacro:macro>
 </robot>

File: denso_robot_descriptions/robots/cobotta/urdf/denso_robot_macro.xacro (robot description, xacro)
@@ -65,5 +65,5 @@
     <gazebo>
       <plugin filename="libgazebo_ros2_control.so" name="gazebo_ros2_control">
-  	<parameters>$(find denso_robot_moveit_config)/robots/$(arg model)/config/denso_robot_controllers.yaml</parameters>
+  	    <parameters>$(find denso_robot_moveit_config)/robots/$(arg model)/config/denso_robot_controllers.yaml</parameters>
       </plugin>
     </gazebo>

File: denso_robot_moveit_config/robots/cobotta/srdf/denso_robot_macro.srdf.xacro (robot description, xacro)
@@ -18,5 +18,10 @@
 		<joint name="$(arg namespace)joint_5"/>
 		<joint name="$(arg namespace)joint_6"/>
-	</group>
+	  </group>
+    <group name="${namespace}hand">
+		<joint name="$(arg namespace)joint_gripper"/>
+		<joint name="$(arg namespace)joint_right_finger"/>
+		<joint name="$(arg namespace)joint_left_finger"/>
+	  </group>
     <!--GROUP STATES - Purpose - Define a named state for a particular group, in terms of joint values. This is useful to define states like 'folded arms'-->
     <!--END EFFECTOR - Purpose - Represent information about an end effector.-->
@@ -32,4 +37,7 @@
 	<disable_collisions link1="$(arg namespace)J3" link2="$(arg namespace)J5" reason="Never"/>
 	<disable_collisions link1="$(arg namespace)J4" link2="$(arg namespace)J5" reason="Adjacent"/>
+	<disable_collisions link1="$(arg namespace)J6" link2="$(arg namespace)gripper_base" reason="Adjacent"/>
+  <disable_collisions link1="$(arg namespace)gripper_base" link2="$(arg namespace)right_finger" reason="Adjacent"/>
+  <disable_collisions link1="$(arg namespace)gripper_base" link2="$(arg namespace)left_finger" reason="Adjacent"/>
   </xacro:macro>
 </robot>

Commit message: Update denso_robot_control

File: denso_robot_descriptions/robots/cobotta/urdf/denso_robot_kinematics.xacro (robot description, xacro)
@@ -271,4 +271,11 @@
 		</joint>
 		<link name="random"/>
+		<joint name="$(arg namespace)joint_tool" type="fixed">
+			<parent link="$(arg namespace)J6"/>
+			<child link="$(arg namespace)tool"/>
+			<origin rpy="0.000000 0.000000 0.000000" xyz="0.000 0.000 0.060"/>
+			<axis xyz="0.000000 0.000000 1.000000"/>
+		</joint>
+		<link name="$(arg namespace)tool" />
 	</xacro:macro>
 </robot>

File: denso_robot_moveit_config/robots/cobotta/srdf/denso_robot_macro.srdf.xacro (robot description, xacro)
@@ -18,4 +18,5 @@
 		<joint name="$(arg namespace)joint_5"/>
 		<joint name="$(arg namespace)joint_6"/>
+		<joint name="$(arg namespace)joint_tool"/>
 	  </group>
     <group name="${namespace}hand">
